File: hardware/KiCad/wire-encoder-modbus-interface.kicad_sch (KiCad schematic)
At the start: 33 parts, among them J1 MODBUS-P1, J2 Programming, J3 MODBUS-P2, J4 Draw-wire, J5 End switch open, J6 End switch close, U1 CH32V003J4M6, U2 MAX3485

Commit message: Final concept PCB-design
Parts:
- added C6: 1n, Capacitor_SMD:C_1206_3216Metric_Pad1.33x1.80mm_HandSolder, symbol Device:C
- added D3: PESD5V0S1BA, Diode_SMD:D_SOD-323_HandSoldering, symbol Device:D_TVS
- added R11: 10k, Resistor_SMD:R_1206_3216Metric_Pad1.30x1.75mm_HandSolder, symbol Device:R
Connections:
- net GND: now also C6.1, D3.1 (A1)
- net WIPER: now also C6.2, D3.2 (A2), R11.1; no longer J4.2 (Pin_2)
- new net: J4.2 (Pin_2), R11.2

Commit message: Some commit in between
Parts:
- removed R10: 470k, Resistor_SMD:R_1206_3216Metric_Pad1.30x1.75mm_HandSolder, symbol Device:R
- R8, R9: value 100k -> 68k
Changed lines of the file:
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@@
 	(wire
 		(pts
-			(xy 223.52 86.36) (xy 223.52 90.17)
-		)
-		(stroke
-			(width 0)
-			(type default)
-		)
-	)
-	(wire
-		(pts
 			(xy 204.47 55.88) (xy 195.58 55.88)
 		)
@@
 	(wire
 		(pts
-			(xy 223.52 97.79) (xy 223.52 101.6)
-		)
-		(stroke
-			(width 0)
-			(type default)
-		)
-	)
-	(wire
-		(pts
 			(xy 220.98 30.48) (xy 201.93 30.48)
 		)
@@
 			)
 		)
-		(property "Value" "100k"
+		(property "Value" "68k"
 			(at 233.172 111.506 90)
 			(show_name no)
@@
 			)
 		)
-	)
-	(symbol
-		(lib_id "Device:R")
-		(at 223.52 93.98 0)
-		(mirror x)
-		(unit 1)
-		(body_style 1)
-		(exclude_from_sim no)
-		(in_bom yes)
-		(on_board yes)
-		(in_pos_files yes)
-		(dnp no)
-		(fields_autoplaced yes)
-		(property "Reference" "R10"
-			(at 220.98 92.7099 0)
-			(show_name no)
-			(do_not_autoplace no)
-			(effects
-				(font
-					(size 1.27 1.27)
-				)
-				(justify right)
-			)
-		)
-		(property "Value" "470k"
-			(at 220.98 95.2499 0)
-			(show_name no)
-			(do_not_autoplace no)
-			(effects
-				(font
-					(size 1.27 1.27)
-				)
-				(justify right)
-			)
-		)
-		(property "Footprint" "Resistor_SMD:R_1206_3216Metric_Pad1.30x1.75mm_HandSolder"
-			(at 221.742 93.98 90)
-			(hide yes)
-			(show_name no)
-			(do_not_autoplace no)
-			(effects
-				(font
-					(size 1.27 1.27)
-				)
-			)
-		)
-		(property "Datasheet" ""
-			(at 223.52 93.98 0)
-			(hide yes)
-			(show_name no)
-			(do_not_autoplace no)
-			(effects
-				(font
-					(size 1.27 1.27)
-				)
-			)
-		)
-		(property "Description" "Resistor"
-			(at 223.52 93.98 0)
-			(hide yes)
-			(show_name no)
-			(do_not_autoplace no)
-			(effects
-				(font
-					(size 1.27 1.27)
-				)
-			)
-		)
-		(pin "1"
-		)
-		(pin "2"
-		)
-		(instances
-			(project "wire-encoder-modbus-interface"
-				(path "/7e9d7b84-ea76-433c-8a90-337ecd1345cc"
-					(reference "R10")
-					(unit 1)
-				)
-			)
-		)
-	)
-	(symbol
+	)	(symbol
 		(lib_id "Connector:Conn_01x03_Pin")
 		(at 250.19 101.6 0)
@@
 			)
 		)
-		(property "Value" "100k"
+		(property "Value" "68k"
 			(at 233.172 104.394 90)
 			(show_name no)
